Commit message: GR_added

File: install/robots_description/share/robots_description/robots/dji_m100.urdf (robot description, URDF)
Before this commit: robot dji_m100, 6 links, 5 joints
Links:
- added link camera_link, mass 0.0010
- link quadrotor: geometry collision cylinder length=0.4 radius=0.35; visual mesh filename=/home/sulieman/quadrotor_target_tracking/src/robots_descrip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
Joints:
- added joint camera_joint: type revolute, parent quadrotor, child camera_link, origin xyz=0 0 0 rpy=0 1.57079633 0, limit lower=0.0 upper=0.0 effort=0 velocity=00.0

Commit message: tracking node added

File: install/robots_description/share/robots_description/robots/dji_m100.urdf (robot description, URDF)
Before this commit: robot dji_m100, 7 links, 6 joints
Links:
- removed link led_link
- link quadrotor: geometry collision cylinder length=0.4 radius=0.35; visual mesh filename=/home/sulieman/quadrotor_target_tracking/install/robots_des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
- link rotor1: geometry 
- link rotor2: geometry 
- link rotor3: geometry 
- link rotor4: geometry 
Joints:
- removed joint led_joint

File: install/robots_description/share/robots_description/robots/ground_robot.xacro (robot description, xacro)
@@ -3,5 +3,5 @@
   <xacro:property name="wheel_radius" value="0.1"/>
   <xacro:property name="wheel_width" value="0.05"/>
-  <xacro:property name="base_width" value="0.5"/>
+  <xacro:property name="base_width" value="0.6"/>
   <xacro:property name="base_length" value="0.8"/>
   <xacro:property name="base_height" value="0.1"/>
@@ -121,5 +121,5 @@
 </gazebo>
 <gazebo reference="base_link">
-  <material>Gazebo/Blue</material>
+  <material>Gazebo/Green</material>
 </gazebo>
 </robot>

File: install/robots_description/share/robots_description/robots/ground_robot.xacro.urdf (robot description, URDF)
Before this commit: robot ground_robot, 6 links, 5 joints
Links:
- link base_link: mass 0.5 -> 1.0; geometry collision box size=0.8 0.6 0.1; visual box size=0.8 0.6 0.1
