Commit message: docker added

File: src/robots_description/robots/dji_m100.urdf (robot description, URDF)
Before this commit: robot dji_m100, 6 links, 5 joints
Links:
- link quadrotor: geometry collision cylinder length=0.4 radius=0.35; visual mesh filename=/root/ros2ws/install/robots_description/share/robots_descri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

File: src/robots_description/robots/ground_robot.xacro (robot description, xacro)
@@ -35,5 +35,5 @@
             <origin rpy="0.0 -1.570796327 0.0" />
             <geometry>
-                <mesh filename="/home/sulieman/quadrotor_target_tracking/src/robots_description/meshes/Marker0.obj" scale="1.0 1.0 1.0" />
+                <mesh filename="$(find robots_description)/meshes/Marker0.obj" scale="1.0 1.0 1.0" />
             </geometry>
         </visual>
@@ -42,5 +42,5 @@
      <parent link="base_link"/>
       <child link="marker"/>
-      <origin xyz="0 -${base_width/2} ${base_height/2+0.01}" rpy="0 0 0"/>
+      <origin xyz="0 -${base_width/2-0.05} ${base_height/2+0.05}" rpy="0 0 0"/>
   </joint>
   <!-- Wheels -->
@@ -120,6 +120,3 @@
     </plugin>
 </gazebo>
-<gazebo reference="base_link">
-  <material>Gazebo/Green</material>
-</gazebo>
 </robot>
